Commit message: Fix persisted central mount and synchronize mobile arm with shared simulation and mission actions

File: models/seer_sba400eu_description/urdf/mobile_manipulator.urdf (robot description, URDF)
Before this commit: robot SEER SBA-400EU + FR5 Mobile Manipulator, 14 links, 13 joints
Links:
- link electrical_cabinet_link: geometry collision box size=.89 .55 .414; visual box size=.002 .060 .039
Joints:
- joint arm_mount_joint: origin xyz=0.31 0 0.426 rpy=0 0 0 -> xyz=0.34 0 0.444 rpy=0 0 0
